File: hardware/control-board/KoloredVerb.kicad_pcb (KiCad board)
At the start: 2 copper layers, 59.6 x 109.5 mm, 51 parts, among them J1 IN, J10 IN, J11 GND, J12 IN, J2 IN, J3 IN, J4 IN, J5 IN, J6 POWER2, J7 IN, J8 IN, J9 POWER1, SW1 SW_Push_Dual, SW2 SW_Push_Dual, SW3 SW_Push_Dual

Commit message: Cut the control board solder mask expansion to 0.0762 mm
Other:
- rule pad_to_mask_clearance: 0.2 -> 0.0762

Commit message: Route the DECAY CV jack to CI4 on the control board
Connections:
- J5 pad T: B5 -> CI4
Routing:
- net B5: track 96.0 -> 0.00 mm
- net CI4: track 0.00 -> 19.2 mm
