File: hardware/core-board/KoloredVerb.core.gates.kicad_sch (KiCad schematic)
At the start: 27 parts, among them U3 4021

Commit message: Drop the core board schematic's leftovers from the trim
Changed lines of the file:
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@@
   (junction (at 68.58 25.4) (diameter 0) (color 0 0 0 0)
-  )
-  (junction (at 35.56 97.79) (diameter 0) (color 0 0 0 0)
-  )
-  (junction (at 135.89 49.53) (diameter 0) (color 0 0 0 0)
   )
   (junction (at 101.6 49.53) (diameter 0) (color 0 0 0 0)
@@
   (junction (at 101.6 25.4) (diameter 0) (color 0 0 0 0)
   )
-  (junction (at 35.56 73.66) (diameter 0) (color 0 0 0 0)
-  )
   (junction (at 135.89 25.4) (diameter 0) (color 0 0 0 0)
   )
   (junction (at 68.58 49.53) (diameter 0) (color 0 0 0 0)
-  )
-  (junction (at 170.18 49.53) (diameter 0) (color 0 0 0 0)
-  )
-  (junction (at 170.18 73.66) (diameter 0) (color 0 0 0 0)
-  )
-  (junction (at 101.6 73.66) (diameter 0) (color 0 0 0 0)
   )
   (junction (at 35.56 25.4) (diameter 0) (color 0 0 0 0)
@@
   (junction (at 35.56 49.53) (diameter 0) (color 0 0 0 0)
   )
-  (junction (at 68.58 73.66) (diameter 0) (color 0 0 0 0)
-  )
-  (junction (at 135.89 73.66) (diameter 0) (color 0 0 0 0)
-  )
   (no_connect (at 241.3 39.37))

Commit message: Verify parts against datasheets, add MPNs, drop stale silkscreen
Parts:
- C5: LCSC (none) -> C14663; MPN (none) -> CC0603KRX7R9BB104
- D1, D2, D3, D4, D5, D6, D7, D8: LCSC (none) -> C22466373; MPN (none) -> BAT54SW
- R1: LCSC (none) -> C21190; MPN (none) -> 0603WAF1001T5E
- R14, R15, R16, R4, R5, R6, R7, R8: LCSC (none) -> C25803; MPN (none) -> 0603WAF1003T5E
- R84, R85, R86, R87, R88, R89, R90, R91: LCSC (none) -> C22935; MPN (none) -> 0603WAF1004T5E
- U3: LCSC (none) -> C2877061; MPN (none) -> CD4021BPWR
Changed lines of the file:
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@@
+      (effects (font (size 1.27 1.27)) hide)
+    )
+    (property "MPN" "CC0603KRX7R9BB104" (id 12) (at 257.81 66.04 0)
+      (effects (font (size 1.27 1.27)) hide)
+    )
+    (property "LCSC" "C14663" (id 13) (at 257.81 66.04 0)
       (effects (font (size 1.27 1.27)) hide)
     )
@@
       (effects (font (size 1.27 1.27)) hide)
     )
+    (property "MPN" "0603WAF1003T5E" (id 12) (at 31.75 20.1422 0)
+      (effects (font (size 1.27 1.27)) hide)
+    )
+    (property "LCSC" "C25803" (id 13) (at 31.75 20.1422 0)
+      (effects (font (size 1.27 1.27)) hide)
+    )
     (pin "1")
     (pin "2")
@@
       (effects (font (size 1.27 1.27)) hide)
     )
+    (property "MPN" "0603WAF1003T5E" (id 12) (at 64.77 20.1422 0)
+      (effects (font (size 1.27 1.27)) hide)
+    )
+    (property "LCSC" "C25803" (id 13) (at 64.77 20.1422 0)
+      (effects (font (size 1.27 1.27)) hide)
+    )
     (pin "1")
     (pin "2")
@@
       (effects (font (size 1.27 1.27)) hide)
     )
+    (property "MPN" "0603WAF1003T5E" (id 12) (at 97.79 20.1422 0)
+      (effects (font (size 1.27 1.27)) hide)
+    )
+    (property "LCSC" "C25803" (id 13) (at 97.79 20.1422 0)
+      (effects (font (size 1.27 1.27)) hide)
+    )
     (pin "1")
     (pin "2")
@@
       (effects (font (size 1.27 1.27)) hide)
     )
+    (property "MPN" "0603WAF1003T5E" (id 12) (at 132.08 20.1422 0)
+      (effects (font (size 1.27 1.27)) hide)
+    )
+    (property "LCSC" "C25803" (id 13) (at 132.08 20.1422 0)
+      (effects (font (size 1.27 1.27)) hide)
+    )
     (pin "1")
     (pin "2")
@@
       (effects (font (size 1.27 1.27)) hide)
     )
+    (property "MPN" "0603WAF1003T5E" (id 12) (at 166.37 20.1422 0)
+      (effects (font (size 1.27 1.27)) hide)
+    )
+    (property "LCSC" "C25803" (id 13) (at 166.37 20.1422 0)
+      (effects (font (size 1.27 1.27)) hide)
+    )
     (pin "1")
     (pin "2")
@@
       (effects (font (size 1.27 1.27)) hide)
     )
+    (property "MPN" "0603WAF1003T5E" (id 12) (at 31.75 44.2722 0)
+      (effects (font (size 1.27 1.27)) hide)
+    )
+    (property "LCSC" "C25803" (id 13) (at 31.75 44.2722 0)
+      (effects (font (size 1.27 1.27)) hide)
+    )
     (pin "1")
     (pin "2")
@@
       (effects (font (size 1.27 1.27)) hide)
     )
+    (property "MPN" "0603WAF1003T5E" (id 12) (at 64.77 44.2722 0)
+      (effects (font (size 1.27 1.27)) hide)
+    )
+    (property "LCSC" "C25803" (id 13) (at 64.77 44.2722 0)
+      (effects (font (size 1.27 1.27)) hide)
+    )
     (pin "1")
     (pin "2")
@@
       (effects (font (size 1.27 1.27)) hide)
     )
+    (property "MPN" "0603WAF1003T5E" (id 12) (at 97.79 44.2722 0)
+      (effects (font (size 1.27 1.27)) hide)
+    )
+    (property "LCSC" "C25803" (id 13) (at 97.79 44.2722 0)
+      (effects (font (size 1.27 1.27)) hide)
+    )
     (pin "1")
     (pin "2")
@@
       (effects (font (size 1.27 1.27)) hide)
     )
+    (property "MPN" "BAT54SW" (id 14) (at 35.56 33.02 0)
+      (effects (font (size 1.27 1.27)) hide)
+    )
+    (property "LCSC" "C22466373" (id 15) (at 35.56 33.02 0)
+      (effects (font (size 1.27 1.27)) hide)
+    )
     (pin "1")
     (pin "2")
@@
       (effects (font (size 1.27 1.27)) hide)
     )
+    (property "MPN" "BAT54SW" (id 14) (at 68.58 33.02 0)
+      (effects (font (size 1.27 1.27)) hide)
+    )
+    (property "LCSC" "C22466373" (id 15) (at 68.58 33.02 0)
+      (effects (font (size 1.27 1.27)) hide)
+    )
     (pin "1")
     (pin "2")
@@
       (effects (font (size 1.27 1.27)) hide)
     )
+    (property "MPN" "BAT54SW" (id 14) (at 101.6 33.02 0)
+      (effects (font (size 1.27 1.27)) hide)
+    )
+    (property "LCSC" "C22466373" (id 15) (at 101.6 33.02 0)
+      (effects (font (size 1.27 1.27)) hide)
+    )
     (pin "1")
     (pin "2")
@@
       (effects (font (size 1.27 1.27)) hide)
     )
+    (property "MPN" "BAT54SW" (id 14) (at 135.89 33.02 0)
+      (effects (font (size 1.27 1.27)) hide)
+    )
+    (property "LCSC" "C22466373" (id 15) (at 135.89 33.02 0)
+      (effects (font (size 1.27 1.27)) hide)
+    )
     (pin "1")
     (pin "2")
@@
       (effects (font (size 1.27 1.27)) hide)
     )
+    (property "MPN" "BAT54SW" (id 14) (at 170.18 33.02 0)
+      (effects (font (size 1.27 1.27)) hide)
+    )
+    (property "LCSC" "C22466373" (id 15) (at 170.18 33.02 0)
+      (effects (font (size 1.27 1.27)) hide)
+    )
     (pin "1")
     (pin "2")
@@
       (effects (font (size 1.27 1.27)) hide)
     )
+    (property "MPN" "BAT54SW" (id 14) (at 35.56 57.15 0)
+      (effects (font (size 1.27 1.27)) hide)
+    )
+    (property "LCSC" "C22466373" (id 15) (at 35.56 57.15 0)
+      (effects (font (size 1.27 1.27)) hide)
+    )
     (pin "1")
     (pin "2")
@@
       (effects (font (size 1.27 1.27)) hide)
     )
+    (property "MPN" "BAT54SW" (id 14) (at 68.58 57.15 0)
+      (effects (font (size 1.27 1.27)) hide)
+    )
+    (property "LCSC" "C22466373" (id 15) (at 68.58 57.15 0)
+      (effects (font (size 1.27 1.27)) hide)
+    )
     (pin "1")
     (pin "2")
@@
       (effects (font (size 1.27 1.27)) hide)
     )
+    (property "MPN" "BAT54SW" (id 14) (at 101.6 57.15 0)
+      (effects (font (size 1.27 1.27)) hide)
+    )
+    (property "LCSC" "C22466373" (id 15) (at 101.6 57.15 0)
+      (effects (font (size 1.27 1.27)) hide)
+    )
     (pin "1")
     (pin "2")
@@
       (effects (font (size 1.27 1.27)) hide)
     )
+    (property "MPN" "0603WAF1004T5E" (id 12) (at 102.87 22.86 0)
+      (effects (font (size 1.27 1.27)) hide)
+    )
+    (property "LCSC" "C22935" (id 13) (at 102.87 22.86 0)
+      (effects (font (size 1.27 1.27)) hide)
+    )
     (pin "1")
     (pin "2")
@@
     )
     (property "Package" "0603" (id 11) (at 68.58 21.59 0)
+      (effects (font (size 1.27 1.27)) hide)
+    )
+    (property "MPN" "0603WAF1004T5E" (id 12) (at 69.85 22.86 0)
+      (effects (font (size 1.27 1.27)) hide)
+    )
+    (property "LCSC" "C22935" (id 13) (at 69.85 22.86 0)
       (effects (font (size 1.27 1.27)) hide)
     )
@@
     )
     (property "ReelRotation" "90" (id 12) (at 231.14 52.07 0)
+      (effects (font (size 1.27 1.27)) hide)
+    )
+    (property "MPN" "CD4021BPWR" (id 13) (at 233.1594 30.5902 0)
+      (effects (font (size 1.27 1.27)) hide)
+    )
+    (property "LCSC" "C2877061" (id 14) (at 233.1594 30.5902 0)
       (effects (font (size 1.27 1.27)) hide)
     )
@@
       (effects (font (size 1.27 1.27)) hide)
     )
+    (property "MPN" "0603WAF1004T5E" (id 12) (at 171.45 22.86 0)
+      (effects (font (size 1.27 1.27)) hide)
+    )
+    (property "LCSC" "C22935" (id 13) (at 171.45 22.86 0)
+      (effects (font (size 1.27 1.27)) hide)
+    )
     (pin "1")
     (pin "2")
@@
       (effects (font (size 1.27 1.27)) hide)
     )
+    (property "MPN" "0603WAF1001T5E" (id 12) (at 209.55 41.91 0)
+      (effects (font (size 1.27 1.27)) hide)
+    )
+    (property "LCSC" "C21190" (id 13) (at 209.55 41.91 0)
+      (effects (font (size 1.27 1.27)) hide)
+    )
     (pin "1")
     (pin "2")
@@
       (effects (font (size 1.27 1.27)) hide)
     )
+    (property "MPN" "0603WAF1004T5E" (id 12) (at 36.83 46.99 0)
+      (effects (font (size 1.27 1.27)) hide)
+    )
+    (property "LCSC" "C22935" (id 13) (at 36.83 46.99 0)
+      (effects (font (size 1.27 1.27)) hide)
+    )
     (pin "1")
     (pin "2")
@@
       (effects (font (size 1.27 1.27)) hide)
     )
+    (property "MPN" "0603WAF1004T5E" (id 12) (at 102.87 46.99 0)
+      (effects (font (size 1.27 1.27)) hide)
+    )
+    (property "LCSC" "C22935" (id 13) (at 102.87 46.99 0)
+      (effects (font (size 1.27 1.27)) hide)
+    )
     (pin "1")
     (pin "2")
@@
       (effects (font (size 1.27 1.27)) hide)
     )
+    (property "MPN" "0603WAF1004T5E" (id 12) (at 69.85 46.99 0)
+      (effects (font (size 1.27 1.27)) hide)
+    )
+    (property "LCSC" "C22935" (id 13) (at 69.85 46.99 0)
+      (effects (font (size 1.27 1.27)) hide)
+    )
     (pin "1")
     (pin "2")
@@
       (effects (font (size 1.27 1.27)) hide)
     )
+    (property "MPN" "0603WAF1004T5E" (id 12) (at 137.16 22.86 0)
+      (effects (font (size 1.27 1.27)) hide)
+    )
+    (property "LCSC" "C22935" (id 13) (at 137.16 22.86 0)
+      (effects (font (size 1.27 1.27)) hide)
+    )
     (pin "1")
     (pin "2")
@@
       (effects (font (size 1.27 1.27)) hide)
     )
+    (property "MPN" "0603WAF1004T5E" (id 12) (at 36.83 22.86 0)
+      (effects (font (size 1.27 1.27)) hide)
+    )
+    (property "LCSC" "C22935" (id 13) (at 36.83 22.86 0)
+      (effects (font (size 1.27 1.27)) hide)
+    )
