File: hardware/core-board/KoloredVerb.core.kicad_pcb (KiCad board)
At the start: 2 copper layers, 59.6 x 109.5 mm, 66 parts, among them J0 POWER BUS, J1 P1, J11 GND, J12 LX2, J2 CIX, J3 BX, J4 LX1, J5 ANALOG, J6 POWER2, J7 BX, J9 POWER1, U1 4051, U3 4021, U6 PCA9685PW

Commit message: Drop the core board schematic's leftovers from the trim
Connections:
- DPSM1 pad D2: /SD_OR_MMC_D3 -> (no net)
- DPSM1 pad D3: /SD_OR_MMC_D2 -> (no net)
- DPSM1 pad D4: /SD_OR_MMC_D1 -> (no net)
- DPSM1 pad D5: /SD_OR_MMC_D0 -> (no net)
- DPSM1 pad D6: /SD_OR_MMC_CLK -> (no net)
- DPSM1 pad D7: /SD_OR_MMC_CMD -> (no net)
Changed lines of the file:
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@@
 			(layers "*.Cu" "*.Mask")
 			(remove_unused_layers no)
-			(net "/SD_OR_MMC_D3")
 			(pinfunction "SDMMC_D3")
 			(pintype "bidirectional")
@@
 			(layers "*.Cu" "*.Mask")
 			(remove_unused_layers no)
-			(net "/SD_OR_MMC_D2")
 			(pinfunction "SDMMC_D2")
 			(pintype "bidirectional")
@@
 			(layers "*.Cu" "*.Mask")
 			(remove_unused_layers no)
-			(net "/SD_OR_MMC_D1")
 			(pinfunction "SDMMC_D1")
 			(pintype "bidirectional")
@@
 			(layers "*.Cu" "*.Mask")
 			(remove_unused_layers no)
-			(net "/SD_OR_MMC_D0")
 			(pinfunction "SDMMC_D0")
 			(pintype "bidirectional")
@@
 			(layers "*.Cu" "*.Mask")
 			(remove_unused_layers no)
-			(net "/SD_OR_MMC_CLK")
 			(pinfunction "SDMMC_CK")
 			(pintype "bidirectional")
@@
 			(layers "*.Cu" "*.Mask")
 			(remove_unused_layers no)
-			(net "/SD_OR_MMC_CMD")
 			(pinfunction "SDMMC_CMD")
 			(pintype "bidirectional")

Commit message: Remove the eurorack-blocks logo from the core board
Parts:
- removed H1: ERB LOGO, Logo_Erb:ErbLog.15mm

Commit message: Verify parts against datasheets, add MPNs, drop stale silkscreen
Other:
- board text added: "KV core r1"
- board text removed: "0..10V"
- board text removed: "Back eMMC"
- board text removed: "CLK"
- board text removed: "CMD"
- board text removed: "D0"
- board text removed: "D1"
- board text removed: "D2"
- board text removed: "D3"
- board text removed: "Front SD"
- board text removed: "SD"
- board text removed: "github.com/ohmtech-rdi/eurorack-blocks"
- board text removed: "rev7"
- board text removed: "±5V"
Changed lines of the file:
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@@
-		)
-	)
-	(gr_text "github.com/ohmtech-rdi/eurorack-blocks"
-		(at 18.28 90.272 0)
-		(layer "F.SilkS")
-		(effects
-			(font
-				(size 1 0.8)
-				(thickness 0.15)
-			)
 		)
 	)
@@
 		)
 	)
-	(gr_text "Back\neMMC"
-		(at 53.205 82.906 0)
-		(layer "F.SilkS")
-		(effects
-			(font
-				(size 1 0.8)
-				(thickness 0.15)
-			)
-		)
-	)
 	(gr_text "L15"
 		(at 53.84 12.675 0)
@@
 		)
 	)
-	(gr_text "Front\nSD"
-		(at 57.269 82.906 0)
-		(layer "F.SilkS")
-		(effects
-			(font
-				(size 1 0.8)
-				(thickness 0.15)
-			)
-		)
-	)
-	(gr_text "SD"
-		(at 55.11 59.03 0)
-		(layer "F.SilkS")
-		(effects
-			(font
-				(size 1 0.8)
-				(thickness 0.15)
-			)
-			(justify right)
-		)
-	)
 	(gr_text "P1"
 		(at 57.65 18.39 0)
@@
 		)
 	)
-	(gr_text "D1"
-		(at 57.65 59.03 0)
-		(layer "F.SilkS")
-		(effects
-			(font
-				(size 1 0.8)
-				(thickness 0.15)
-			)
-			(justify right)
-		)
-	)
-	(gr_text "D0"
-		(at 57.65 61.57 0)
-		(layer "F.SilkS")
-		(effects
-			(font
-				(size 1 0.8)
-				(thickness 0.15)
-			)
-			(justify right)
-		)
-	)
-	(gr_text "CLK"
-		(at 57.65 64.11 0)
-		(layer "F.SilkS")
-		(effects
-			(font
-				(size 1 0.8)
-				(thickness 0.15)
-			)
-			(justify right)
-		)
-	)
-	(gr_text "CMD"
-		(at 57.65 66.65 0)
-		(layer "F.SilkS")
-		(effects
-			(font
-				(size 1 0.8)
-				(thickness 0.15)
-			)
-			(justify right)
-		)
-	)
-	(gr_text "D3"
-		(at 57.65 69.19 0)
-		(layer "F.SilkS")
-		(effects
-			(font
-				(size 1 0.8)
-				(thickness 0.15)
-			)
-			(justify right)
-		)
-	)
-	(gr_text "D2"
-		(at 57.65 71.73 0)
-		(layer "F.SilkS")
-		(effects
-			(font
-				(size 1 0.8)
-				(thickness 0.15)
-			)
-			(justify right)
-		)
-	)
 	(gr_text "GND"
 		(at 57.65 97.13 0)
@@
 		)
 	)
-	(gr_text "0..10V"
-		(at 38.219 99.162 0)
-		(layer "F.SilkS")
-		(effects
-			(font
-				(size 1 0.9)
-				(thickness 0.15)
-			)
-			(justify left)
-		)
-	)
-	(gr_text "±5V"
-		(at 38.219 97.638 0)
-		(layer "F.SilkS")
-		(effects
-			(font
-				(size 1 1)
-				(thickness 0.15)
-			)
-			(justify left)
-		)
-	)
-	(gr_text "CI1"
-		(at 46.22 97.13 0)
-		(layer "F.SilkS")
-		(effects
-			(font
-				(size 1 1)
-				(thickness 0.15)
-			)
-			(justify right)
-		)
-	)
-	(gr_text "CI2"
-		(at 46.22 99.67 0)
-		(layer "F.SilkS")
-		(effects
-			(font
-				(size 1 1)
-				(thickness 0.15)
-			)
-			(justify right)
-		)
-	)
-	(gr_text "rev7"
+	(gr_text "KV core r1"
 		(at 53.5 117.5 0)
 		(layer "F.SilkS")
