File: hardware/core-board/KoloredVerb.core.kicad_sch (KiCad schematic)
At the start: 21 parts, among them J1 P1, J11 GND, J12 LX2, J2 CIX, J3 BX, J4 LX1, J5 ANALOG, J6 POWER2, J7 BX, J9 POWER1

Commit message: Drop the core board schematic's leftovers from the trim
Connections:
- net SD_OR_MMC_CLK: no longer names the net of DPSM1.D6 (SDMMC_CK)
- net SD_OR_MMC_CMD: no longer names the net of DPSM1.D7 (SDMMC_CMD)
- net SD_OR_MMC_D0: no longer names the net of DPSM1.D5 (SDMMC_D0)
- net SD_OR_MMC_D1: no longer names the net of DPSM1.D4 (SDMMC_D1)
- net SD_OR_MMC_D2: no longer names the net of DPSM1.D3 (SDMMC_D2)
- net SD_OR_MMC_D3: no longer names the net of DPSM1.D2 (SDMMC_D3)
- no-connect marks 1 -> 7
Other:
- note added: "Just needed for BOM They are: - 4x 2x5 female socket for the DPSM - 1x 1x36 Male header"
- note removed: "Just needed for BOM They are: - 4x 2x5 female socket for the DPSM - 1x 1x36 Male header - 8x Jumpers"
Changed lines of the file:
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@@
   (paper "A4")
   (no_connect (at 176.53 26.67))
-  (text "Just needed for BOM\nThey are:\n- 4x 2x5 female socket for the DPSM\n- 1x 1x36 Male header\n- 8x Jumpers"
+  (text "Just needed for BOM\nThey are:\n- 4x 2x5 female socket for the DPSM\n- 1x 1x36 Male header"
     (at 246.38 57.15 0)
     (effects (font (size 1.27 1.27)) (justify left bottom))
@@
     (effects (font (size 1.27 1.27)) (justify left bottom))
   )
-  (label "SD_OR_MMC_CLK" (at 158.75 57.15 180)
-    (effects (font (size 1.27 1.27)) (justify right bottom))
-  )
   (label "ADC1_MUX" (at 50.8 116.84 0)
     (effects (font (size 1.27 1.27)) (justify left bottom))
@@
     (effects (font (size 1.27 1.27)) (justify left bottom))
   )
-  (label "SD_OR_MMC_D0" (at 158.75 62.23 180)
-    (effects (font (size 1.27 1.27)) (justify right bottom))
-  )
   (label "GATE_SR_LATCH" (at 158.75 82.55 180)
     (effects (font (size 1.27 1.27)) (justify right bottom))
   )
-  (label "SD_OR_MMC_D1" (at 158.75 64.77 180)
-    (effects (font (size 1.27 1.27)) (justify right bottom))
-  )
-  (label "SD_OR_MMC_CMD" (at 158.75 59.69 180)
-    (effects (font (size 1.27 1.27)) (justify right bottom))
-  )
   (label "ADC_MUX_ADDR_C" (at 31.75 154.94 180)
     (effects (font (size 1.27 1.27)) (justify right bottom))
@@
   )
   (label "ADC_MUX_ADDR_C" (at 158.75 85.09 180)
-    (effects (font (size 1.27 1.27)) (justify right bottom))
-  )
-  (label "SD_OR_MMC_D2" (at 158.75 67.31 180)
-    (effects (font (size 1.27 1.27)) (justify right bottom))
-  )
-  (label "SD_OR_MMC_D3" (at 158.75 69.85 180)
     (effects (font (size 1.27 1.27)) (justify right bottom))
   )
@@
     (pin "1")
   )
+  (no_connect (at 158.75 57.15))
+  (no_connect (at 158.75 59.69))
+  (no_connect (at 158.75 62.23))
+  (no_connect (at 158.75 64.77))
+  (no_connect (at 158.75 67.31))
+  (no_connect (at 158.75 69.85))
 )

Commit message: Remove the eurorack-blocks logo from the core board
Parts:
- removed H1: ERB LOGO, Logo_Erb:ErbLog.15mm, symbol Mechanical:MountingHole
Changed lines of the file:
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@@
     (pin "1")
-  )
-  (symbol (lib_id "Mechanical:MountingHole") (at 251.46 91.44 0) (unit 1)
-    (in_bom yes) (on_board yes)
-    (property "Reference" "H1" (id 0) (at 254 90.2716 0)
-      (effects (font (size 1.27 1.27)) (justify left))
-    )
-    (property "Value" "ERB LOGO" (id 1) (at 254 92.583 0)
-      (effects (font (size 1.27 1.27)) (justify left))
-    )
-    (property "Footprint" "Logo_Erb:ErbLog.15mm" (id 2) (at 251.46 91.44 0)
-      (effects (font (size 1.27 1.27)) hide)
-    )
-    (property "Datasheet" "~" (id 3) (at 251.46 91.44 0)
-      (effects (font (size 1.27 1.27)) hide)
-    )
   )
   (symbol (lib_id "power:GND") (at 107.95 175.26 90) (unit 1)
@@
       (reference "Dummy5") (unit 1) (value "Big Pin Header") (footprint "Empty:Empty")
     )
-    (path "/00000000-0000-0000-0000-0000609ea577"
-      (reference "H1") (unit 1) (value "ERB LOGO") (footprint "Logo_Erb:ErbLog.15mm")
-    )
     (path "/c55c6a2b-7145-443e-a402-9d8950328d23"

Commit message: Verify parts against datasheets, add MPNs, drop stale silkscreen
Parts:
- D30: LCSC (none) -> C22466373; MPN (none) -> BAT54SW
- DPSM1: MPN (none) -> DAISY-PATCH-SM
- Dummy1, Dummy2, Dummy3, Dummy4: MPN (none) -> PPPC052LFBN-RC
- Dummy5: MPN (none) -> PBC36SAAN
- J1: MPN (none) -> PPTC121LFBN-RC
- J11, J9: MPN (none) -> PPTC021LFBN-RC
- J12, J3, J4, J7: MPN (none) -> PPTC081LFBN-RC
- J2: MPN (none) -> PPTC091LFBN-RC
- J5: MPN (none) -> PPTC101LFBN-RC
- J6: MPN (none) -> PPTC041LFBN-RC
Changed lines of the file:
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@@
+      (effects (font (size 1.27 1.27)) hide)
+    )
+    (property "MPN" "DAISY-PATCH-SM" (id 4) (at 182.88 58.42 0)
       (effects (font (size 1.27 1.27)) hide)
     )
@@
       (effects (font (size 1.27 1.27)) hide)
     )
+    (property "MPN" "PPTC091LFBN-RC" (id 11) (at 104.14 21.59 0)
+      (effects (font (size 1.27 1.27)) hide)
+    )
     (pin "1")
     (pin "2")
@@
     )
     (property "DistLink" "https://www.digikey.de/en/products/detail/sullins-connector-solutions/PPTC121LFBN-RC/807231" (id 10) (at 26.67 39.37 0)
+      (effects (font (size 1.27 1.27)) hide)
+    )
+    (property "MPN" "PPTC121LFBN-RC" (id 11) (at 27.94 21.59 0)
       (effects (font (size 1.27 1.27)) hide)
     )
@@
       (effects (font (size 1.27 1.27)) hide)
     )
+    (property "MPN" "PPTC021LFBN-RC" (id 11) (at 54.61 81.28 0)
+      (effects (font (size 1.27 1.27)) hide)
+    )
     (pin "1")
     (pin "2")
@@
     )
     (property "DistLink" "https://www.digikey.de/en/products/detail/sullins-connector-solutions/PPTC041LFBN-RC/810144" (id 10) (at 76.2 57.15 0)
+      (effects (font (size 1.27 1.27)) hide)
+    )
+    (property "MPN" "PPTC041LFBN-RC" (id 11) (at 78.74 49.53 0)
       (effects (font (size 1.27 1.27)) hide)
     )
@@
       (effects (font (size 1.27 1.27)) hide)
     )
+    (property "MPN" "PPTC021LFBN-RC" (id 11) (at 29.21 69.85 0)
+      (effects (font (size 1.27 1.27)) hide)
+    )
     (pin "1")
     (pin "2")
@@
     )
     (property "DistLink" "https://www.digikey.de/product-detail/en/sullins-connector-solutions/PPTC081LFBN-RC/S7006-ND/810147" (id 10) (at 53.34 34.29 0)
+      (effects (font (size 1.27 1.27)) hide)
+    )
+    (property "MPN" "PPTC081LFBN-RC" (id 11) (at 55.88 21.59 0)
       (effects (font (size 1.27 1.27)) hide)
     )
@@
       (effects (font (size 1.27 1.27)) hide)
     )
+    (property "MPN" "PPTC081LFBN-RC" (id 11) (at 78.74 21.59 0)
+      (effects (font (size 1.27 1.27)) hide)
+    )
     (pin "1")
     (pin "2")
@@
       (effects (font (size 1.27 1.27)) hide)
     )
+    (property "MPN" "PPTC081LFBN-RC" (id 11) (at 55.88 49.53 0)
+      (effects (font (size 1.27 1.27)) hide)
+    )
     (pin "1")
     (pin "2")
@@
       (effects (font (size 1.27 1.27)) hide)
     )
+    (property "MPN" "PPTC081LFBN-RC" (id 11) (at 78.74 67.31 0)
+      (effects (font (size 1.27 1.27)) hide)
+    )
     (pin "1")
     (pin "2")
@@
     )
     (property "DistLink" "https://www.digikey.de/en/products/detail/sullins-connector-solutions/PPTC101LFBN-RC/810149" (id 10) (at 120.65 34.29 0)
+      (effects (font (size 1.27 1.27)) hide)
+    )
+    (property "MPN" "PPTC101LFBN-RC" (id 11) (at 123.19 19.05 0)
       (effects (font (size 1.27 1.27)) hide)
     )
@@
     (property "DistLink" "https://www.digikey.de/en/products/detail/sullins-connector-solutions/PPPC052LFBN-RC/810245" (id 10) (at 228.6 43.18 0)
       (effects (font (size 1.27 1.27)) hide)
+    )    (property "MPN" "PPPC052LFBN-RC" (id 11) (at 231.14 42.0116 0)
+      (effects (font (size 1.27 1.27)) hide)
     )
   )
@@
     (property "DistLink" "https://www.digikey.de/en/products/detail/sullins-connector-solutions/PPPC052LFBN-RC/810245" (id 10) (at 228.6 48.26 0)
       (effects (font (size 1.27 1.27)) hide)
+    )    (property "MPN" "PPPC052LFBN-RC" (id 11) (at 231.14 47.0916 0)
+      (effects (font (size 1.27 1.27)) hide)
     )
   )
@@
     (property "DistLink" "https://www.digikey.de/en/products/detail/sullins-connector-solutions/PPPC052LFBN-RC/810245" (id 10) (at 228.6 53.34 0)
       (effects (font (size 1.27 1.27)) hide)
+    )    (property "MPN" "PPPC052LFBN-RC" (id 11) (at 231.14 52.1716 0)
+      (effects (font (size 1.27 1.27)) hide)
     )
   )
@@
     (property "DistLink" "https://www.digikey.de/en/products/detail/sullins-connector-solutions/PPPC052LFBN-RC/810245" (id 10) (at 228.6 58.42 0)
       (effects (font (size 1.27 1.27)) hide)
+    )    (property "MPN" "PPPC052LFBN-RC" (id 11) (at 231.14 57.2516 0)
+      (effects (font (size 1.27 1.27)) hide)
     )
   )
@@
     )
     (property "DistLink" "https://www.digikey.de/en/products/detail/sullins-connector-solutions/PBC36SAAN/859621" (id 10) (at 228.6 64.77 0)
+      (effects (font (size 1.27 1.27)) hide)
+    )    (property "MPN" "PBC36SAAN" (id 11) (at 231.14 63.6016 0)
       (effects (font (size 1.27 1.27)) hide)
     )
@@
       (effects (font (size 1.27 1.27)) hide)
     )
+    (property "MPN" "BAT54SW" (id 14) (at 118.11 73.66 0)
+      (effects (font (size 1.27 1.27)) hide)
+    )
+    (property "LCSC" "C22466373" (id 15) (at 118.11 73.66 0)
+      (effects (font (size 1.27 1.27)) hide)
+    )
