File: hardware/core-board/KoloredVerb.core.leds.kicad_sch (KiCad schematic)
At the start: 9 parts, among them U6 PCA9685PW

Commit message: Verify parts against datasheets, add MPNs, drop stale silkscreen
Parts:
- C8: LCSC (none) -> C14663; MPN (none) -> CC0603KRX7R9BB104
- R47, R48, R49, R50, R51: LCSC (none) -> C21190; MPN (none) -> 0603WAF1001T5E
- R79, R80: LCSC (none) -> C23162; MPN (none) -> 0603WAF4701T5E
- U6: LCSC (none) -> C2678753; MPN (none) -> PCA9685PW
Changed lines of the file:
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@@
+      (effects (font (size 1.27 1.27)) hide)
+    )
+    (property "MPN" "0603WAF1001T5E" (id 12) (at 114.3 85.09 0)
+      (effects (font (size 1.27 1.27)) hide)
+    )
+    (property "LCSC" "C21190" (id 13) (at 114.3 85.09 0)
       (effects (font (size 1.27 1.27)) hide)
     )
@@
       (effects (font (size 1.27 1.27)) hide)
     )
+    (property "MPN" "0603WAF1001T5E" (id 12) (at 114.3 87.63 0)
+      (effects (font (size 1.27 1.27)) hide)
+    )
+    (property "LCSC" "C21190" (id 13) (at 114.3 87.63 0)
+      (effects (font (size 1.27 1.27)) hide)
+    )
     (pin "1")
     (pin "2")
@@
       (effects (font (size 1.27 1.27)) hide)
     )
+    (property "MPN" "0603WAF1001T5E" (id 12) (at 114.3 90.17 0)
+      (effects (font (size 1.27 1.27)) hide)
+    )
+    (property "LCSC" "C21190" (id 13) (at 114.3 90.17 0)
+      (effects (font (size 1.27 1.27)) hide)
+    )
     (pin "1")
     (pin "2")
@@
       (effects (font (size 1.27 1.27)) hide)
     )
+    (property "MPN" "0603WAF1001T5E" (id 12) (at 114.3 92.71 0)
+      (effects (font (size 1.27 1.27)) hide)
+    )
+    (property "LCSC" "C21190" (id 13) (at 114.3 92.71 0)
+      (effects (font (size 1.27 1.27)) hide)
+    )
     (pin "1")
     (pin "2")
@@
       (effects (font (size 1.27 1.27)) hide)
     )
+    (property "MPN" "0603WAF1001T5E" (id 12) (at 114.3 95.25 0)
+      (effects (font (size 1.27 1.27)) hide)
+    )
+    (property "LCSC" "C21190" (id 13) (at 114.3 95.25 0)
+      (effects (font (size 1.27 1.27)) hide)
+    )
     (pin "1")
     (pin "2")
@@
       (effects (font (size 1.27 1.27)) hide)
     )
+    (property "MPN" "0603WAF4701T5E" (id 12) (at 143.51 49.3522 0)
+      (effects (font (size 1.27 1.27)) hide)
+    )
+    (property "LCSC" "C23162" (id 13) (at 143.51 49.3522 0)
+      (effects (font (size 1.27 1.27)) hide)
+    )
     (pin "1")
     (pin "2")
@@
     )
     (property "JlcPcbPartNumber" "C23162" (id 11) (at 143.51 64.77 0)
+      (effects (font (size 1.27 1.27)) hide)
+    )
+    (property "MPN" "0603WAF4701T5E" (id 12) (at 143.51 59.5122 0)
+      (effects (font (size 1.27 1.27)) hide)
+    )
+    (property "LCSC" "C23162" (id 13) (at 143.51 59.5122 0)
       (effects (font (size 1.27 1.27)) hide)
     )
@@
     )
     (property "JlcPcbPartNumber" "C2678753" (id 11) (at 88.9 96.52 0)
+      (effects (font (size 1.27 1.27)) hide)
+    )
+    (property "MPN" "PCA9685PW" (id 12) (at 97.79 121.92 0)
+      (effects (font (size 1.27 1.27)) hide)
+    )
+    (property "LCSC" "C2678753" (id 13) (at 97.79 121.92 0)
       (effects (font (size 1.27 1.27)) hide)
     )
@@
       (effects (font (size 1.27 1.27)) hide)
     )
+    (property "MPN" "CC0603KRX7R9BB104" (id 12) (at 102.87 63.5 0)
+      (effects (font (size 1.27 1.27)) hide)
+    )
+    (property "LCSC" "C14663" (id 13) (at 102.87 63.5 0)
+      (effects (font (size 1.27 1.27)) hide)
+    )
