File: hardware/core-board/KoloredVerb.core.pots.kicad_sch (KiCad schematic)
At the start: 2 parts, among them U1 4051

Commit message: Verify parts against datasheets, add MPNs, drop stale silkscreen
Parts:
- C3: LCSC (none) -> C14663; MPN (none) -> CC0603KRX7R9BB104
- U1: LCSC (none) -> C54587; MPN (none) -> CD4051BPWR
Changed lines of the file:
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@@
+      (effects (font (size 1.27 1.27)) hide)
+    )
+    (property "MPN" "CD4051BPWR" (id 13) (at 123.19 100.33 0)
+      (effects (font (size 1.27 1.27)) hide)
+    )
+    (property "LCSC" "C54587" (id 14) (at 123.19 100.33 0)
       (effects (font (size 1.27 1.27)) hide)
     )
@@
       (effects (font (size 1.27 1.27)) hide)
     )
+    (property "MPN" "CC0603KRX7R9BB104" (id 12) (at 139.7 106.68 0)
+      (effects (font (size 1.27 1.27)) hide)
+    )
+    (property "LCSC" "C14663" (id 13) (at 139.7 106.68 0)
+      (effects (font (size 1.27 1.27)) hide)
+    )
