File: hardware/core-board/KoloredVerb.core.power.kicad_sch (KiCad schematic)
At the start: 7 parts, among them J0 POWER BUS

Commit message: Verify parts against datasheets, add MPNs, drop stale silkscreen
Parts:
- C1, C2: LCSC (none) -> C15850; MPN (none) -> CL21A106KAYNNNE
- D23, D24: LCSC (none) -> C8598; MPN (none) -> B5819W SL
- J0: MPN (none) -> 61201021621
- L1, L2: LCSC (none) -> C85824; MPN (none) -> BLM18AG102SN1D
Changed lines of the file:
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@@
+      (effects (font (size 1.27 1.27)) hide)
+    )
+    (property "MPN" "BLM18AG102SN1D" (id 12) (at 171.45 83.2104 0)
+      (effects (font (size 1.27 1.27)) hide)
+    )
+    (property "LCSC" "C85824" (id 13) (at 171.45 83.2104 0)
       (effects (font (size 1.27 1.27)) hide)
     )
@@
       (effects (font (size 1.27 1.27)) hide)
     )
+    (property "MPN" "B5819W SL" (id 13) (at 158.75 84.6836 0)
+      (effects (font (size 1.27 1.27)) hide)
+    )
+    (property "LCSC" "C8598" (id 14) (at 158.75 84.6836 0)
+      (effects (font (size 1.27 1.27)) hide)
+    )
     (pin "1")
     (pin "2")
@@
       (effects (font (size 1.27 1.27)) hide)
     )
+    (property "MPN" "B5819W SL" (id 13) (at 158.75 105.0036 0)
+      (effects (font (size 1.27 1.27)) hide)
+    )
+    (property "LCSC" "C8598" (id 14) (at 158.75 105.0036 0)
+      (effects (font (size 1.27 1.27)) hide)
+    )
     (pin "1")
     (pin "2")
@@
       (effects (font (size 1.27 1.27)) hide)
     )
+    (property "MPN" "BLM18AG102SN1D" (id 12) (at 171.45 103.5304 0)
+      (effects (font (size 1.27 1.27)) hide)
+    )
+    (property "LCSC" "C85824" (id 13) (at 171.45 103.5304 0)
+      (effects (font (size 1.27 1.27)) hide)
+    )
     (pin "1")
     (pin "2")
@@
     )
     (property "DistLink" "https://www.digikey.de/product-detail/en/würth-elektronik/61201021621/732-2094-ND/2060590" (id 9) (at 119.38 101.6 0)
+      (effects (font (size 1.27 1.27)) hide)
+    )
+    (property "MPN" "61201021621" (id 10) (at 120.65 91.0082 0)
       (effects (font (size 1.27 1.27)) hide)
     )
@@
       (effects (font (size 1.27 1.27)) hide)
     )
+    (property "MPN" "CL21A106KAYNNNE" (id 12) (at 185.801 105.5116 0)
+      (effects (font (size 1.27 1.27)) hide)
+    )
+    (property "LCSC" "C15850" (id 13) (at 185.801 105.5116 0)
+      (effects (font (size 1.27 1.27)) hide)
+    )
     (pin "1")
     (pin "2")
@@
       (effects (font (size 1.27 1.27)) hide)
     )
+    (property "MPN" "CL21A106KAYNNNE" (id 12) (at 185.801 92.8116 0)
+      (effects (font (size 1.27 1.27)) hide)
+    )
+    (property "LCSC" "C15850" (id 13) (at 185.801 92.8116 0)
+      (effects (font (size 1.27 1.27)) hide)
+    )
